File: kicad_files/hardware_challenge.kicad_sch (KiCad schematic)
At the start: 25 parts, among them J1 12V INPUT, J3 Cable header, Q1 SiSS27DN, SW1 TEST BUTTON, U1 L7805, U2 Teensy4.1, U3 NEO-M8N, U4 CY8C9560A-24AXIT, U5 MAX2679

Commit message: Fix firmware and schematic bugs from harness tester challenge
Firmware (firmware.ino, CY8C9560.*):
- Fix inverted start-button logic
- Fix pass/fail logic (require all 40 pins to match, not just one)
- Fix 32-bit shift overflow in per-pin bitmask calculation
- Fix expander bit-to-harness-pin mapping (bits 20-23 are SCL/SDA, not GPIO)
- Add missing pinMode(OUTPUT) for GPS SAFEBOOT/RESET lines
- Add bounds check on NMEA receive buffer
- Fix CY8C9560 reset sequence to actually release RESET_N before I2C use
- Add I2C error tracking to the CY8C9560 driver
- Add debounce/single-shot logic so a test only runs once per button press

Schematic (hardware_challenge.kicad_sch):
- Fix R3 (I2C SDA pull-up) wired to GND instead of +3.3V
- Fix NEO-M8N VDD_USB wired to GND instead of +3.3V
- Mirror Q1 so the reverse-polarity MOSFET's Source/Drain face the
  correct sides (Source to raw input, Drain to protected rail)
- Add R5/R6/R7 series resistors for the RGB status LED
- Add R8/R9 pull-ups on GPS SAFEBOOT/RESET lines

All changes verified with kicad-cli sch erc and netlist export after
each edit; no new ERC violations introduced. PCB layout bugs (wrong
U4 footprint, unrouted D3 pad, trace-width/clearance violations, etc.)
are not fixed here since the new resistors have no PCB footprint yet -
that requires KiCad's GUI-only "Update PCB from Schematic" step.

Co-Authored-By: Claude <noreply@anthropic.com>
Parts:
- added R5, R6, R7: 330, Resistor_SMD:R_0402_1005Metric, symbol Device:R
- added R8, R9: 10k, Resistor_SMD:R_0402_1005Metric, symbol Device:R
Connections:
- net +12V: now also Q1.5 (D); no longer Q1.1 (S), Q1.2 (S), Q1.3 (S)
- net +3.3V: now also R3.1, U3.7 (VDD_USB), R8.1, R9.1
- net GND: no longer R3.1, U3.7 (VDD_USB)
- net LED_B: now also U2.7 (5_IN2), U2.8 (6_OUT1D), R5.1, R6.1, R7.1; no longer D3.2 (BK)
- net UBX-RST_N: now also R9.2
- net UBX-SAFEBOOT: now also R8.2
- net at D1.1 (A1), J1.1: now also Q1.1 (S), Q1.2 (S), Q1.3 (S); no longer Q1.5 (D)
- net LED_G: no longer names the net of D3.3 (GK)
- net LED_G: now also R6.2; no longer U2.8 (6_OUT1D)
- net LED_R: no longer names the net of D3.4 (RK)
- net LED_R: now also R5.2; no longer U2.7 (5_IN2)
- new net: D3.2 (BK), R7.2
